File: totoro-pcb-macropad.kicad_pcb (KiCad board)
At the start: 2 copper layers, 57.2 x 78.7 mm, 37 parts, among them J1 USB4085-GF-A_REVA, SW1 SW_PUSH, U1 ATMEGA32U4, X1 XTAL_GND

Commit message: PCB layout
Parts:
- moved SW1 104.3 mm to (215.4, 34.3)
- moved C1 72.2 mm to (180.0, 32.0), turned to 270 degrees
- moved X1 65.6 mm to (175.6, 32.0), turned to 180 degrees
- moved C6 64.4 mm to (183.5, 37.4)
- moved F1 63.3 mm to (193.9, 40.2), turned to 90 degrees
- moved R4 60.9 mm to (188.3, 40.2)
- moved R3 60.9 mm to (190.5, 40.2)
- moved C2 59.1 mm to (171.3, 32.0), turned to 270 degrees
- moved C5 57.2 mm to (167.6, 37.0), turned to 90 degrees
- moved C8 53.3 mm to (183.5, 41.6), turned to 270 degrees
- moved U1 50.0 mm to (175.5, 41.4), turned to 180 degrees
- moved C7 47.5 mm to (183.5, 45.9), turned to 270 degrees
- moved R5 46.4 mm to (199.5, 40.2), turned to 90 degrees
- moved C3 40.7 mm to (180.5, 49.3), turned to 0 degrees
- moved R6 39.5 mm to (197.4, 40.2), turned to 270 degrees
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Connections:
- C1 pad 2: +5V -> GND
- C2 pad 2: +5V -> GND
- C3 pad 1: VCC -> +5V
- C3 pad 2: +5V -> GND
- C4 pad 1: VCC -> +5V
- C4 pad 2: +5V -> GND
- C5 pad 1: VCC -> +5V
- C5 pad 2: +5V -> GND
- C6 pad 1: VCC -> +5V
- C6 pad 2: +5V -> GND
- C7 pad 1: VCC -> +5V
- C7 pad 2: +5V -> GND
- C8 pad 2: +5V -> GND
- J1 pad A1: +5V -> GND
- J1 pad A12: +5V -> GND
- J1 pad B1: +5V -> GND
- J1 pad B12: +5V -> GND
- J1 pad P1: +5V -> GND
- J1 pad P2: +5V -> GND
- J1 pad P3: +5V -> GND
- J1 pad P4: +5V -> GND
- R1 pad 2: VCC -> +5V
- R2 pad 1: +5V -> GND
- R5 pad 1: +5V -> GND
- R6 pad 2: +5V -> GND
- SW1 pad 1: +5V -> GND
- U1 pad 14: VCC -> +5V
- U1 pad 15: +5V -> GND
- U1 pad 23: +5V -> GND
- U1 pad 24: VCC -> +5V
- U1 pad 34: VCC -> +5V
- U1 pad 35: +5V -> GND
- U1 pad 43: +5V -> GND
- U1 pad 44: VCC -> +5V
- U1 pad 5: +5V -> GND
- X1 pad 3: +5V -> GND
Routing:
- net GND: track 0.00 -> 59.3 mm
- net Net-(R1-Pad1): track 0.00 -> 47.8 mm
- net +5V: track 0.00 -> 14.5 mm
- net Net-(J1-PadB5): track 0.00 -> 13.7 mm, vias 0 -> 1
- net VCC: track 0.00 -> 12.5 mm
- net Net-(J1-PadA7): track 0.00 -> 10.2 mm
- net Net-(C2-Pad1): track 0.00 -> 9.31 mm
- net Net-(C1-Pad1): track 0.00 -> 9.17 mm
- net Net-(J1-PadA6): track 0.00 -> 8.63 mm
- net Net-(J1-PadA5): track 0.00 -> 6.08 mm, vias 0 -> 2
- net Net-(C8-Pad1): track 0.00 -> 2.26 mm
- net Net-(R2-Pad2): track 0.00 -> 1.85 mm
- added copper zone on B.Cu, net GND
- added copper zone on F.Cu, net GND
Other:
- board size 57.2 x 78.7 mm -> 57.2 x 79.2 mm
- net class Default: trace_width 0.25 -> 0.3
- net class Power added: clearance 0.2, trace_width 0.4, via_dia 0.8, via_drill 0.4

Commit message: Final commit
Parts:
- added G***: LOGO, totoro-pcb-macropad:toto-img, F.Cu at (207.0, 42.4)
-  : renamed from F1
-  : renamed from R1
-  : renamed from J1
-  : renamed from D9
-  : renamed from D8
-  : renamed from D7
-  : renamed from D6
-  : renamed from D5
-  : renamed from D4
-  : renamed from D3
-  : renamed from D2
-  : renamed from X1
-  : renamed from D1
-  : renamed from C8
-  : renamed from C7
-  : renamed from C6
-  : renamed from C5
-  : renamed from C4
-  : renamed from C3
-  : renamed from C2
-  : renamed from C1
-  : renamed from U1
-  : renamed from SW1
-  : renamed from R6
-  : renamed from R5
-  : renamed from R4
-  : renamed from R3
-  : renamed from R2
- moved   0.46 mm to (183.5, 41.2)
Connections:
-   pad 36: Net-(U1-Pad36) -> ROW2
-   pad 37: Net-(U1-Pad37) -> ROW1
-   pad 38: Net-(U1-Pad38) -> ROW0
-   pad 39: Net-(U1-Pad39) -> COL0
-   pad 40: Net-(U1-Pad40) -> COL1
-   pad 41: Net-(U1-Pad41) -> COL2
Routing:
- net ROW2: track 0.00 -> 112.0 mm, vias 0 -> 1
- net ROW1: track 0.00 -> 92.6 mm, vias 0 -> 1
- net COL2: track 0.00 -> 77.6 mm
- net ROW0: track 0.00 -> 73.2 mm, vias 0 -> 1
- net +5V: track 14.5 -> 83.0 mm, vias 0 -> 4
- net COL1: track 0.00 -> 59.3 mm
- net COL0: track 0.00 -> 50.3 mm
- net GND: track 59.3 -> 81.2 mm
- net Net-(D2-Pad2): track 0.00 -> 11.0 mm
- net Net-(D8-Pad2): track 0.00 -> 11.0 mm
- net Net-(D7-Pad2): track 0.00 -> 11.0 mm
- net Net-(D9-Pad2): track 0.00 -> 11.0 mm
- net Net-(D5-Pad2): track 0.00 -> 10.9 mm
- net Net-(D3-Pad2): track 0.00 -> 10.9 mm
- net Net-(D1-Pad2): track 0.00 -> 10.9 mm
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Other:
- board text added: "Esche 2020"

Commit message: Probably fix crystal footprint, but i dont remember
Parts:
- moved   53.8 mm to (124.8, 59.2)
- moved   53.8 mm to (147.4, 67.4)
- moved   53.8 mm to (137.0, 59.2)
- moved   53.8 mm to (147.1, 58.0)
- moved   53.8 mm to (166.2, 131.4)
- moved   53.8 mm to (147.2, 131.4)
- moved   53.8 mm to (128.1, 131.4)
- moved   53.8 mm to (166.2, 112.4)
- moved   53.8 mm to (147.2, 112.4)
- moved   53.8 mm to (128.1, 112.4)
- moved   53.8 mm to (166.2, 93.3)
- moved   53.8 mm to (147.2, 93.3)
- moved   53.8 mm to (129.2, 59.2)
- moved   53.8 mm to (128.1, 93.3)
- moved   53.8 mm to (137.0, 68.4)
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